File: Lightbar.kicad_sch (KiCad schematic)
At the start: 20 parts, among them IC1 PAM2863ECR, IC2 PAM2863ECR, J1 Conn_01x04_Pin, Q1 2N2219

Commit message: Add note
Added note for min current for LEDs
Other:
- note added: "Note: Vin = 5V @ 3A (min)"
Changed lines of the file:
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@@
 (kicad_sch
-	(version 20231120)
+	(version 20250114)
 	(generator "eeschema")
-	(generator_version "8.0")
+	(generator_version "9.0")
 	(paper "User" 317.5 254.127)
+	(text "PWM"
+		(exclude_from_sim no)
+		(at 142.24 167.64 0)
+		(effects
+			(font
+				(size 1.778 1.5113)
+			)
+			(justify left bottom)
+		)
+	)
+	(text "PWM"
+		(exclude_from_sim no)
+		(at 142.24 88.9 0)
+		(effects
+			(font
+				(size 1.778 1.5113)
+			)
+			(justify left bottom)
+		)
+	)
+	(text "Note:\nVin = 5V @ 3A (min)"
+		(exclude_from_sim no)
+		(at 86.106 40.132 0)
+		(effects
+			(font
+				(size 1.27 1.27)
+			)
+			(justify left)
+		)
+	)
 	(junction
 		(at 82.55 156.21)
@@
 			(width 0.1524)
 			(type solid)
-		)
-	)
-	(text "PWM"
-		(exclude_from_sim no)
-		(at 142.24 167.64 0)
-		(effects
-			(font
-				(size 1.778 1.5113)
-			)
-			(justify left bottom)
-		)
-	)
-	(text "PWM"
-		(exclude_from_sim no)
-		(at 142.24 88.9 0)
-		(effects
-			(font
-				(size 1.778 1.5113)
-			)
-			(justify left bottom)
 		)
 	)
@@
 		)
 	)
+	(embedded_fonts no)
 )
